Commit message: Add files via upload

File: vehicle_description/urdf/truck_step2.urdf (robot description, URDF)
Before this commit: robot truck, 2 links, 1 joints
Links:
- link chassis: geometry collision mesh filename=package://vehicle_description/meshes/truck/truck_step2.stl scale=0.00001 0.00001 0.00001; visual mesh filename=package://vehicle_description/meshes/truck/truck_step2.stl scale=0.00001 0.00001 0.00001

File: vehicle_description/urdf/truck_step3.urdf (robot description, URDF)
Before this commit: robot truck, 2 links, 1 joints
Links:
- link chassis: geometry collision mesh filename=package://vehicle_description/meshes/truck/truck_step3.stl scale=0.00001 0.00001 0.00001; visual mesh filename=package://vehicle_description/meshes/truck/truck_step3.stl scale=0.00001 0.00001 0.00001
