Commit message: add revolute

File: lds_data/urdf/lds_revolute.urdf.xacro (robot description, xacro)
@@ -14,5 +14,5 @@
     <origin xyz="0 0 0" rpy="0 0 0"/>
     <axis xyz="0 1 0"/>
-    <limit lower="-1.570796" upper="1.570796" effort="11" velocity="0.0348"/>
+    <limit lower="-3.14159" upper="3.14159" effort="100" velocity="0.17453278"/>
   </joint>
   <transmission name="sick5xx_revolute_tran">
